File: board_53.kicad_pcb (KiCad board)
At the start: 4 copper layers, 43.2 x 17.8 mm, 18 parts, among them J1 Analog, J2 Digital, J4 USB_B_Micro, SW1 RESET, SW2 BTN1, U1 MDBT53-1M

Commit message: Init commit
Parts:
- removed D1: RED_LED, LED_SMD:LED_0805_2012Metric_Pad1.15x1.40mm_HandSolder
- removed D2: GREEN_LED, LED_SMD:LED_0805_2012Metric_Pad1.15x1.40mm_HandSolder
- removed J4: USB_B_Micro, Connector_USB:USB_Micro-B_Amphenol_10118193-0001LF_Horizontal
- removed R6: 2.2, Resistor_SMD:R_0805_2012Metric_Pad1.20x1.40mm_HandSolder
- added C3: GRM188R60J106ME47D, Capacitor_SMD:C_0603_1608Metric_Pad1.08x0.95mm_HandSolder, F.Cu at (110.8, 92.9)
- added C4: CL10A105KQ8NNNC, Capacitor_SMD:C_0603_1608Metric_Pad1.08x0.95mm_HandSolder, F.Cu at (126.5, 94.6)
- added D3: LTST-C19HE1WT, LED_SMD:LED_LiteOn_LTST-C19HE1WT, F.Cu at (111.5, 88.0)
- added J3: 12402012E212A, 12402012E212A:AMPHENOL_12402012E212A, F.Cu at (101.6, 91.1)
- added L1: WIP201612S-2R2MLDG, Inductor_SMD:L_0805_2012Metric_Pad1.15x1.40mm_HandSolder, F.Cu at (113.4, 94.8)
- added L2: MLZ1608N100LT000, Inductor_SMD:L_0603_1608Metric_Pad1.05x0.95mm_HandSolder, F.Cu at (126.5, 96.2)
- added L3: MLZ1608N100LT000, Inductor_SMD:L_0603_1608Metric_Pad1.05x0.95mm_HandSolder, F.Cu at (134.7, 97.0)
- added R1: ERJ-2RKF3300X, Resistor_SMD:R_0402_1005Metric_Pad0.72x0.64mm_HandSolder, F.Cu at (113.9, 87.6)
- added R7: ERJ-2GEJ512X, Resistor_SMD:R_0402_1005Metric_Pad0.72x0.64mm_HandSolder, F.Cu at (107.8, 88.5)
- added U2: TPS62291DRVR, Package_SON:WSON-6-1EP_2x2mm_P0.65mm_EP1x1.6mm_ThermalVias, F.Cu at (110.9, 95.0)
- C1: value 2.2uF -> CL10A105KQ8NNNC; footprint Capacitor_SMD:C_0805_2012Metric_Pad1.18x1.45mm_HandSolder -> Capacitor_SMD:C_0603_1608Metric_Pad1.08x0.95mm_HandSolder
- C2: value 4.7uF -> GRM188R60J106ME47D; footprint Capacitor_SMD:C_0805_2012Metric_Pad1.18x1.45mm_HandSolder -> Capacitor_SMD:C_0603_1608Metric_Pad1.08x0.95mm_HandSolder
- R3: value 1M -> ERJ-2GEJ512X; footprint Resistor_SMD:R_0805_2012Metric_Pad1.20x1.40mm_HandSolder -> Resistor_SMD:R_0402_1005Metric_Pad0.72x0.64mm_HandSolder
- R4, R5: value 330R -> ERJ-2RKF3300X; footprint Resistor_SMD:R_0805_2012Metric_Pad1.20x1.40mm_HandSolder -> Resistor_SMD:R_0402_1005Metric_Pad0.72x0.64mm_HandSolder
- SW1: value RESET -> CS1213AGF160
- SW2: value BTN1 -> CS1213AGF160
- moved C2 15.4 mm to (108.4, 94.6), turned to -90 degrees
- moved C1 11.9 mm to (138.1, 97.0), turned to 0 degrees
- moved R3 6.75 mm to (108.8, 88.5)
- moved R5 5.05 mm to (113.9, 88.9), turned to 0 degrees
- moved R4 4.19 mm to (113.9, 86.3), turned to 0 degrees
- moved SW2 1.25 mm to (121.8, 93.7), turned to 90 degrees
- moved SW1 0.49 mm to (121.8, 88.0), turned to -90 degrees
Connections:
- C1 pad 1: +3V3 -> Net-(U1A-DECR)
- C2 pad 1: VBUS_CL -> VBUS
- R3 pad 1: Net-(J4-Shield) -> GND
- R3 pad 2: GND -> Net-(J3-CC1_B)
- R5 pad 2: /GR_LED -> /BL_LED
- U1 pad 41: VBUS_CL -> +3V3
- U1 pad 44: VBUS_CL -> VBUS
- U1 pad 50: unconnected-(U1A-DCCD-Pad50) -> Net-(U1A-DCCD)
- U1 pad 52: unconnected-(U1A-DECD-Pad52) -> Net-(U1A-DECD)
- U1 pad 54: unconnected-(U1A-DCC-Pad54) -> Net-(U1A-DCC)
- U1 pad 58: unconnected-(U1A-DECR-Pad58) -> Net-(U1A-DECR)
- U1 pad 60: /GR_LED -> /BL_LED
- U1 pad 65: /P0.29 -> /GR_LED
Routing:
- net /BL_LED: track 0.00 -> 28.5 mm, vias 0 -> 2
- net VBUS_CL: track 25.1 -> 0.00 mm
- net VBUS: track 19.2 -> 43.7 mm, vias 0 -> 1
- net GND: track 12.8 -> 34.7 mm
- net Net-(J4-Shield): track 14.8 -> 0.00 mm
- net Net-(U1A-DECD): track 0.00 -> 12.0 mm
- net Net-(U1A-DCCD): track 0.00 -> 7.24 mm
- net Net-(J3-CC1_B): track 0.00 -> 5.66 mm
- net /P0.16: track 6.89 -> 11.1 mm
- net /~{RESET}: track 22.5 -> 18.4 mm, vias 2 -> 0
- net /RD_LED: track 26.9 -> 30.7 mm
- net Net-(U1A-DECR): track 0.00 -> 3.75 mm
- net +3V3: track 34.8 -> 37.5 mm
- net /GR_LED: track 26.9 -> 24.3 mm
- net Net-(U1A-DCC): track 0.00 -> 2.25 mm
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Other:
- board text added: "github.com/ ffenix113/board_53"
- board text added: "v0.1"
- board text added: "vbus"
- board text removed: "0.02"
- board text removed: "VBUS"
- board text removed: "github.com/ ffenix113/ zigbee_home"
- board text removed: "v0.0"
