File: board_53.kicad_sch (KiCad schematic)
At the start: 14 parts, among them J1 Analog, J2 Digital, J4 USB_B_Micro, SW1 RESET, SW2 BTN1, U1 MDBT53-1M

Commit message: Init commit
Parts:
- removed D1: RED_LED, LED_SMD:LED_0805_2012Metric_Pad1.15x1.40mm_HandSolder, symbol Device:LED
- removed D2: GREEN_LED, LED_SMD:LED_0805_2012Metric_Pad1.15x1.40mm_HandSolder, symbol Device:LED
- removed J4: USB_B_Micro, Connector_USB:USB_Micro-B_Amphenol_10118193-0001LF_Horizontal, symbol Connector:USB_B_Micro
- removed R6: 2.2, Resistor_SMD:R_0805_2012Metric_Pad1.20x1.40mm_HandSolder, symbol Device:R
- added C3: GRM188R60J106ME47D, Capacitor_SMD:C_0603_1608Metric_Pad1.08x0.95mm_HandSolder, symbol Device:C_Small
- added C4: CL10A105KQ8NNNC, Capacitor_SMD:C_0603_1608Metric_Pad1.08x0.95mm_HandSolder, symbol Device:C_Small
- added D3: LTST-C19HE1WT, LED_SMD:LED_LiteOn_LTST-C19HE1WT, symbol LTST-C19HE1WT:LTST-C19HE1WT
- added J3: 12402012E212A, 12402012E212A:AMPHENOL_12402012E212A, symbol 12402012E212A:12402012E212A
- added L1: WIP201612S-2R2MLDG, Inductor_SMD:L_0805_2012Metric_Pad1.15x1.40mm_HandSolder, symbol Device:L
- added L2, L3: MLZ1608N100LT000, Inductor_SMD:L_0603_1608Metric_Pad1.05x0.95mm_HandSolder, symbol Device:L
- added R1: ERJ-2RKF3300X, Resistor_SMD:R_0402_1005Metric_Pad0.72x0.64mm_HandSolder, symbol Device:R
- added R7: ERJ-2GEJ512X, Resistor_SMD:R_0402_1005Metric_Pad0.72x0.64mm_HandSolder, symbol Device:R
- added U2: TPS62291DRVR, Package_SON:WSON-6-1EP_2x2mm_P0.65mm_EP1x1.6mm_ThermalVias, symbol TPS62291DRVR:TPS62291DRVR
- C1: value 2.2uF -> CL10A105KQ8NNNC; footprint Capacitor_SMD:C_0805_2012Metric_Pad1.18x1.45mm_HandSolder -> Capacitor_SMD:C_0603_1608Metric_Pad1.08x0.95mm_HandSolder
- C2: value 4.7uF -> GRM188R60J106ME47D; footprint Capacitor_SMD:C_0805_2012Metric_Pad1.18x1.45mm_HandSolder -> Capacitor_SMD:C_0603_1608Metric_Pad1.08x0.95mm_HandSolder
- R3: value 1M -> ERJ-2GEJ512X; footprint Resistor_SMD:R_0805_2012Metric_Pad1.20x1.40mm_HandSolder -> Resistor_SMD:R_0402_1005Metric_Pad0.72x0.64mm_HandSolder
- R4, R5: value 330R -> ERJ-2RKF3300X; footprint Resistor_SMD:R_0805_2012Metric_Pad1.20x1.40mm_HandSolder -> Resistor_SMD:R_0402_1005Metric_Pad0.72x0.64mm_HandSolder
- SW1: value RESET -> CS1213AGF160
- SW2: value BTN1 -> CS1213AGF160
Connections:
- net P0.29 is gone; now on net GR_LED: U1.65 (P0.29)
- net +3V3: now also U1.41 (VDDH), C3.1, D3.4, L1.2, U2.3 (FB); no longer C1.1
- net +5V: now also C2.1, U1.44 (VBUS), J3.A4_B9 (VBUS), J3.B4_A9 (VBUS__1), U2.4 (EN), U2.5 (VIN)
- net GND: now also R3.1, C3.2, C4.1, J3.A1_B12 (GND), J3.B1_A12 (GND__1), J3.SH1 (SHIELD), J3.SH2 (SHIELD__1), J3.SH3 (SHIELD__2), J3.SH4 (SHIELD__3), R7.2, U2.2 (MODE), U2.6 (GND); no longer R3.2
- net GR_LED: now also R1.2; no longer R5.2, U1.60 (P0.28)
- net USB_DN: now also J3.A7 (D-_A), J3.B7 (D-_B)
- net USB_DP: now also J3.A6 (D+_A), J3.B6 (D+_B)
- net at R4.1: now also D3.1
- net at R5.1: now also D3.3
- net at U1.50 (DCCD): now also L2.2
- net at U1.52 (DECD): now also C4.2, L2.1
- net at U1.54 (DCC): now also L3.2
- net at U1.58 (DECR): now also C1.1, L3.1
- removed net VBUS_CL: C2.1, U1.41 (VDDH), U1.44 (VBUS)
- new net: L1.1, U2.1 (SW)
- new net: J3.A5 (CC1_A), R7.1
- new net: J3.B5 (CC1_B), R3.2
- new net: D3.2, R1.1
- new net BL_LED: R5.2, U1.60 (P0.28)
- no-connect marks 8 -> 6
Other:
- moved on the sheet: C2, R4, U1A

Commit message: add schematic pdf
Parts:
- C1, C4: value CL10A105KQ8NNNC -> 1uF
- C2, C3: value GRM188R60J106ME47D -> 10uF
- R1, R4, R5: value ERJ-2RKF3300X -> 330 Ohm
- R3, R7: value ERJ-2GEJ512X -> 5.1 kOhm
